Commit message: adding lidar frame

File: src/robots/go2w_description/urdf/go2w_description.urdf (robot description, URDF)
Before this commit: robot go2w_description, 34 links, 33 joints
Links:
- added link lidar_frame, mass 0
Joints:
- added joint lidar_joint: type fixed, parent trunk, child lidar_frame, origin xyz=0.0 0.0 0.1 rpy=0 0 0, axis 0 0 0

File: src/robots/go2w_description/xacro/lidar.xacro (robot description, xacro)
@@ -1,5 +1,5 @@
 <?xml version="1.0"?>
 <robot xmlns:xacro="http://www.ros.org/wiki/xacro" >
-    <gazebo reference="radar_link">
+    <gazebo reference="lidar_frame">
         <material>Gazebo/Red</material>
         <sensor type="ray" name="velodyne2-HDL32E">
@@ -38,5 +38,5 @@
               <remapping>~/out:=point_cloud</remapping>
             </ros>
-            <frame_name>radar_link</frame_name>
+            <frame_name>lidar_frame</frame_name>
             <organize_cloud>false</organize_cloud>
             <min_range>0.9</min_range>

Commit message: add velodyne vlp 16 and reduce speed for joy

File: src/robots/go2w_description/urdf/go2w_description.urdf (robot description, URDF)
Before this commit: robot go2w_description, 35 links, 34 joints
Links:
- link lidar_frame: mass 0 -> None; geometry visual mesh filename=package://velodyne_description/meshes/VLP16_scan.dae
Joints:
- joint imu_joint: origin xyz=-0.02557 0 0.04232 rpy=0 0 0 -> xyz=0 0 0 rpy=0 0 0

File: src/robots/go2w_description/xacro/lidar.xacro (robot description, xacro)
@@ -2,6 +2,47 @@
 <robot xmlns:xacro="http://www.ros.org/wiki/xacro" >
     <gazebo reference="lidar_frame">
-        <material>Gazebo/Red</material>
-        <sensor type="ray" name="velodyne2-HDL32E">
+        <sensor name="velodyne-VLP16" type="ray">
+            <pose>0 0 0 0 0 0</pose>
+            <visualize>false</visualize>
+            <update_rate>10</update_rate>
+            <ray>
+                <scan>
+                <horizontal>
+                    <samples>440</samples>
+                    <resolution>1</resolution>
+                    <min_angle>-3.141592653589793</min_angle>
+                    <max_angle>3.141592653589793</max_angle>
+                </horizontal>
+                <vertical>
+                    <samples>16</samples>
+                    <resolution>1</resolution>
+                    <min_angle>-0.2617993877991494</min_angle>
+                    <max_angle>
+                        0.2617993877991494</max_angle>
+                </vertical>
+                </scan>
+                <range>
+                <min>0.3</min>
+                <max>131.0</max>
+                <resolution>0.001</resolution>
+                </range>
+                <noise>
+                <type>gaussian</type>
+                <mean>0.0</mean>
+                <stddev>0.0</stddev>
+                </noise>
+            </ray>
+            <plugin filename="libgazebo_ros_velodyne_laser.so" name="gazebo_ros_laser_controller">
+                <ros>
+                    <namespace>/unitree_go2w/lidar</namespace>
+                    <remapping>~/out:=point_cloud</remapping>
+                </ros>
+                <frameName>lidar_frame</frameName>
+                <min_range>0.9</min_range>
+                <max_range>130.0</max_range>
+                <gaussianNoise>0.008</gaussianNoise>
+            </plugin>
+        </sensor>
+        <!-- <sensor type="ray" name="velodyne2-HDL32E">
           <pose>0 0 0 0 0 0</pose>
           <visualize>false</visualize>
@@ -44,5 +85,5 @@
             <gaussian_noise>0.008</gaussian_noise>
           </plugin>
-        </sensor>
+        </sensor> -->
     </gazebo>
 </robot>

Commit message: add support for mid360

File: src/robots/go2w_description/urdf/go2w_description.urdf (robot description, URDF)
Before this commit: robot go2w_description, 35 links, 34 joints
Links:
- link lidar_frame: geometry 

File: src/robots/go2w_description/xacro/lidar-vlp16.xacro (robot description, xacro)
@@ -44,46 +44,4 @@
             </plugin>
         </sensor>
-        <!-- <sensor type="ray" name="velodyne2-HDL32E">
-          <pose>0 0 0 0 0 0</pose>
-          <visualize>false</visualize>
-          <update_rate>10</update_rate>
-          <ray>
-                <scan>
-                    <horizontal>
-                        <samples>220</samples>
-                        <resolution>1</resolution>
-                        <min_angle>-3.142</min_angle>
-                        <max_angle>3.142</max_angle>
-                    </horizontal>
-                    <vertical>
-                        <samples>32</samples>
-                        <resolution>1</resolution>
-                        <min_angle>-0.535</min_angle>
-                        <max_angle> 0.186</max_angle>
-                    </vertical>
-                </scan>
-                <range>
-                    <min>0.3</min>
-                    <max>131.0</max>
-                    <resolution>0.001</resolution>
-                </range>
-                <noise>
-                    <type>gaussian</type>
-                    <mean>0.0</mean>
-                    <stddev>0.0</stddev>
-                </noise>
-          </ray>
-          <plugin name="gazebo_ros_laser_controller" filename="libgazebo_ros_velodyne_laser.so">
-            <ros>
-              <namespace>/unitree_go2w/lidar</namespace>
-              <remapping>~/out:=point_cloud</remapping>
-            </ros>
-            <frame_name>lidar_frame</frame_name>
-            <organize_cloud>false</organize_cloud>
-            <min_range>0.9</min_range>
-            <max_range>130.0</max_range>
-            <gaussian_noise>0.008</gaussian_noise>
-          </plugin>
-        </sensor> -->
     </gazebo>
 </robot>

File: src/robots/go2w_description/xacro/robot.xacro (robot description, xacro)
@@ -3,5 +3,5 @@
     <xacro:include filename="$(find go2w_description)/urdf/go2w_description.urdf"/>
     <xacro:include filename="$(find go2w_description)/xacro/gazebo.xacro"/>
-    <xacro:include filename="$(find go2w_description)/xacro/lidar.xacro"/>
+    <xacro:include filename="$(find go2w_description)/xacro/lidar-mid360.xacro"/>
     <xacro:include filename="$(find go2w_description)/xacro/camera.xacro"/>
 </robot>

Commit message: gt pose publishing

File: src/robots/go2w_description/urdf/go2w_description.urdf (robot description, URDF)
Before this commit: robot go2w_description, 35 links, 34 joints
Links:
- link lidar_frame: mass None -> 0

File: src/robots/go2w_description/xacro/gazebo.xacro (robot description, xacro)
@@ -227,4 +227,21 @@
         </plugin>
     </gazebo>
+    <!-- <gazebo>
+        <plugin name="p3d_base_controller" filename="libgazebo_ros_p3d.so">
+            <alwaysOn>true</alwaysOn>
+            <updateRate>50.0</updateRate>
+            <bodyName>robot_model</bodyName>
+            <topicName>ground_truth/state</topicName>
+            <gaussianNoise>0.01</gaussianNoise>
+            <frameName>world</frameName>
+            <xyzOffsets>0 0 0</xyzOffsets>
+            <rpyOffsets>0 0 0</rpyOffsets>
+        </plugin>
+        <plugin name="gazebo_ros_state" filename="libgazebo_ros_state.so">
+            <update_rate>50</update_rate>
+            <publish_model_states>true</publish_model_states>
+            <publish_link_states>true</publish_link_states>
+        </plugin>
+    </gazebo> -->
     </xacro:if>
     <gazebo reference="base">

File: src/robots/go2w_description/xacro/lidar-mid360.xacro (robot description, xacro)
@@ -2,5 +2,5 @@
 <robot xmlns:xacro="http://www.ros.org/wiki/xacro" >
     <xacro:include filename="$(find ros2_livox_simulation)/urdf/mid360.xacro"/>
-    <xacro:mid360 name="livox" parent="base" topic="unitree_go2w/lidar">
+    <xacro:mid360 name="livox_frame" parent="base" topic="unitree_go2w/lidar">
         <origin xyz="0 0 0.1" rpy="0 0 0"/>
     </xacro:mid360>
